Commit message: fix URDF

File: elite_description/urdf/ec66_description_real.urdf (robot description, URDF)
Before this commit: robot ec66, 9 links, 8 joints
Joints:
- joint joint2: limit lower=-3.14 upper=0 effort=150.0 velocity=2.61993 -> lower=-6.2832 upper=6.2832 effort=150.0 velocity=2.61993
- joint joint3: origin xyz=0 0.418 0 rpy=0 0 1.10 -> xyz=0 0.418 0 rpy=0 0 1.5708
