Commit message: 1. reorganized and changed file names 2. made the elite arm xacro modular and compatible for both ec66 and cs66(yet to be added) 3. added initial positions for arm

File: elite_description/urdf/elite_description.urdf.xacro (robot description, xacro)
@@ -1,46 +1,33 @@
-<?xml version="1.0" ?>
-<robot xmlns:xacro="http://www.ros.org/wiki/xacro" name="ec66">
+<?xml version="1.0"?>
+<robot xmlns:xacro="http://www.ros.org/wiki/xacro" name="elite">
     <!-- Set use_gazebo = false for implementation on real rover -->
     <xacro:arg name="use_gazebo" default="false"/>
-    <xacro:arg name="arm_type" default="ec66"/>
+    <xacro:arg name="arm" default="ec66"/>
+    <xacro:arg name="use_moveit" default="false"/>
     <!-- Include macros -->
-    <xacro:include filename="$(find elite_description)/urdf/macro/elite_macro.urdf.xacro" />
-    <!-- World Link and Joint -->
-    <link name="world" />
-    <joint name="world_joint" type="fixed">
+    <xacro:include filename="$(find elite_description)/urdf/macro/elite_macro.xacro" />
+    <!--Elite arm parameters-->
+    <xacro:arg name="arm_parent" default="world"/>
+    <xacro:arg name="tf_prefix" default=""/>
+    <xacro:arg name="joint_limit_params_file" default="$(find elite_description)/config/$(arg arm)/joint_limits.yaml"/>
+    <xacro:arg name="joint_origin_params_file" default="$(find elite_description)/config/$(arg arm)/joint_origins.yaml"/>
+    <xacro:arg name="link_inertials_params_file" default="$(find elite_description)/config/$(arg arm)/link_inertials.yaml"/>
+    <xacro:arg name="initial_joint_positions_file" default="$(find elite_description)/config/$(arg arm)/initial_positions.yaml"/>
+    <!--create arm-->
+    <xacro:elite_robot
+        name="$(arg arm)"
+        tf_prefix="$(arg tf_prefix)"
+        arm_parent="$(arg arm_parent)"
+        joint_limits_parameters_file="$(arg joint_limit_params_file)"
+        joint_origins_parameters_file="$(arg joint_origin_params_file)"
+        link_inertials_parameters_file="$(arg link_inertials_params_file)"
+    >
         <origin xyz="0 0 0" rpy="0 0 0" />
-        <parent link="world" />
-        <child link="base_link" />
-    </joint>
-    <!-- Base Link -->
-    <xacro:link_macro name="base_link" />
-    <!-- Link1 and Joint1 -->
-    <xacro:link_macro name="link1" />
-    <xacro:joint_macro name="joint1" />
-    <!-- Link2 and Joint2 -->
-    <xacro:link_macro name="link2" />
-    <xacro:joint_macro name="joint2" />
-    <!-- Link3 and Joint3 -->
-    <xacro:link_macro name="link3" />
-    <xacro:joint_macro name="joint3" />
-    <!-- Link4 and Joint4 -->
-    <xacro:link_macro name="link4" />
-    <xacro:joint_macro name="joint4" />
-    <!-- Link5 and Joint5 -->
-    <xacro:link_macro name="link5" />
-    <xacro:joint_macro name="joint5" />
-    <!-- Link6 and Joint6 -->
-    <xacro:link_macro name="link6" />
-    <xacro:joint_macro name="joint6" />
-    <!-- Flange -->
-    <link name="flange" />
-    <joint name="flange_joint" type="fixed">
-        <origin xyz="0 0 0" rpy="0 0 0" />
-        <parent link="link6" />
-        <child link="flange" />
-    </joint>
-    <!-- Include ros2_control configuration for simulation -->
-    <xacro:if value="$(arg use_gazebo)">
-        <xacro:include filename="$(find elite_description)/urdf/elite_gazebo_ros2_control.urdf.xacro" />
-    </xacro:if>
+    </xacro:elite_robot>
+    <xacro:unless value="$(arg use_moveit)">
+        <!-- Include ros2_control configuration for simulation -->
+        <xacro:if value="$(arg use_gazebo)">
+            <xacro:include filename="$(find elite_description)/urdf/elite_gazebo_ros2_control.urdf.xacro" />
+        </xacro:if>
+    </xacro:unless>
 </robot>

File: elite_description/urdf/elite_gazebo_ros2_control.urdf.xacro (robot description, xacro)
@@ -1,13 +1,14 @@
 <?xml version="1.0" ?>
-<robot xmlns:xacro="http://www.ros.org/wiki/xacro" name="ec66">
-    <xacro:include filename="$(find elite_description)/urdf/macro/elite_ros2_control_macro.urdf.xacro" />
+<robot xmlns:xacro="http://www.ros.org/wiki/xacro" name="elite">
+    <xacro:include filename="$(find elite_description)/urdf/macro/elite_ros2_control_macro.xacro" />
     <!-- Use the ros2_control_macro with individual joints -->
     <xacro:ros2_control_macro
         name="GazeboSystem"
         plugin="gazebo_ros2_control/GazeboSystem"
-        parameters="$(find elite_gazebo)/config/$(arg arm_type)_ros2_control.yaml" />
+        parameters="$(find elite_gazebo)/config/$(arg arm)_ros2_control.yaml"
+        tf_prefix="$(arg tf_prefix)" />
     <!-- Use the gazebo_macro -->
     <xacro:gazebo_macro
         filename="libgazebo_ros2_control.so"
-        parameters="$(find elite_gazebo)/config/$(arg arm_type)_ros2_control.yaml" />
+        parameters="$(find elite_gazebo)/config/$(arg arm)_ros2_control.yaml" />
 </robot>

File: elite_description/urdf/macro/elite_common.xacro (robot description, xacro)
@@ -3,16 +3,16 @@
   <!-- Load parameters from YAML files -->
   <xacro:property
-    name="config_joint_limits"
-    value="${xacro.load_yaml('$(find elite_description)/config/$(arg arm_type)/joint_limits_ec66.yaml')}"/>
+    name="joint_limits_parameters"
+    value="${xacro.load_yaml('$(arg joint_limit_params_file)')}"/>
   <xacro:property
-    name="config_joint_origins"
-    value="${xacro.load_yaml('$(find elite_description)/config/$(arg arm_type)/joint_origins_ec66.yaml')}"/>
+    name="joint_origins_parameters"
+    value="${xacro.load_yaml('$(arg joint_origin_params_file)')}"/>
   <xacro:property
-    name="config_link_inertials"
-    value="${xacro.load_yaml('$(find elite_description)/config/$(arg arm_type)/link_inertials_ec66.yaml')}"/>
+    name="link_inertials_parameters"
+    value="${xacro.load_yaml('$(arg link_inertials_params_file)')}"/>
   <!-- Extract subsections from yaml dictionaries -->
-  <xacro:property name="joint_limits" value="${config_joint_limits['joint_limits']}"/>
-  <xacro:property name="joint_origins" value="${config_joint_origins['joint_origins']}"/>
-  <xacro:property name="link_inertials" value="${config_link_inertials['link_inertials']}"/>
+  <xacro:property name="joint_limits" value="${joint_limits_parameters['joint_limits']}"/>
+  <xacro:property name="joint_origins" value="${joint_origins_parameters['joint_origins']}"/>
+  <xacro:property name="link_inertials" value="${link_inertials_parameters['link_inertials']}"/>
   <!-- Define macros using loaded parameters -->
   <xacro:macro name="link_macro" params="name">

File: elite_description/urdf/macro/elite_ros2_control_macro.xacro (robot description, xacro)
@@ -3,4 +3,11 @@
     <xacro:property name="min_val" value="-3.15"/>
     <xacro:property name="max_val" value="3.15"/>
+    <!-- Load parameters from YAML file -->
+    <xacro:property
+        name="initial_positions_params"
+        value="${xacro.load_yaml('$(arg initial_joint_positions_file)')}"
+    />
+    <!-- Extract subsections from yaml dictionaries -->
+    <xacro:property name="initial_positions" value="${initial_positions_params['initial_positions']}"/>
     <!-- Macro for defining joint interfaces -->
     <xacro:macro name="joint_interface_macro" params="joint_name">
@@ -14,5 +21,8 @@
             <param name="max">${max_val}</param>
         </command_interface>
-        <state_interface name="position"/>
+        <state_interface name="position">
+            <!-- initial position for the mock system and simulation -->
+            <param name="initial_value">${initial_positions[joint_name]}</param>
+        </state_interface>
         <state_interface name="velocity"/>
         <state_interface name="effort"/>
@@ -20,5 +30,5 @@
     </xacro:macro>
     <!-- Macro for ROS2 Control Configuration -->
-    <xacro:macro name="ros2_control_macro" params="name plugin parameters">
+    <xacro:macro name="ros2_control_macro" params="name plugin parameters tf_prefix">
         <ros2_control name="${name}" type="system">
         <hardware>
@@ -27,10 +37,10 @@
         </hardware>
         <!-- Directly instantiate each joint interface -->
-        <xacro:joint_interface_macro joint_name="joint1"/>
-        <xacro:joint_interface_macro joint_name="joint2"/>
-        <xacro:joint_interface_macro joint_name="joint3"/>
-        <xacro:joint_interface_macro joint_name="joint4"/>
-        <xacro:joint_interface_macro joint_name="joint5"/>
-        <xacro:joint_interface_macro joint_name="joint6"/>
+        <xacro:joint_interface_macro joint_name="${tf_prefix}joint1"/>
+        <xacro:joint_interface_macro joint_name="${tf_prefix}joint2"/>
+        <xacro:joint_interface_macro joint_name="${tf_prefix}joint3"/>
+        <xacro:joint_interface_macro joint_name="${tf_prefix}joint4"/>
+        <xacro:joint_interface_macro joint_name="${tf_prefix}joint5"/>
+        <xacro:joint_interface_macro joint_name="${tf_prefix}joint6"/>
         </ros2_control>
     </xacro:macro>

File: elite_moveit/config/ec66.urdf.xacro (robot description, xacro)
@@ -2,8 +2,8 @@
 <robot xmlns:xacro="http://www.ros.org/wiki/xacro" name="ec66">
     <xacro:arg name="initial_positions_file" default="initial_positions.yaml" />
+    <xacro:arg name="arm" default="ec66"/>
+    <xacro:arg name="use_moveit" default="true"/>
     <!-- Import elite_description urdf file with arm_type argument -->
-    <xacro:include filename="$(find elite_description)/urdf/elite_description.urdf.xacro">
-        <xacro:arg name="arm_type" value="ec66"/>
-    </xacro:include>
+    <xacro:include filename="$(find elite_description)/urdf/elite_description.urdf.xacro"/>
     <!-- Import control_xacro -->
     <xacro:include filename="ec66.ros2_control.xacro" />

File: elite_moveit/config/ec66_simulation.urdf.xacro (robot description, xacro)
@@ -2,10 +2,10 @@
 <robot xmlns:xacro="http://www.ros.org/wiki/xacro" name="ec66">
     <xacro:arg name="initial_positions_file" default="initial_positions.yaml" />
+    <xacro:arg name="use_gazebo" value="true"/>
+    <xacro:arg name="arm" value="ec66"/>
     <!-- Import ec66 urdf file with use_gazebo set to true -->
-    <xacro:include filename="$(find elite_description)/urdf/ec66_description.urdf.xacro">
-        <xacro:arg name="use_gazebo" value="true"/>
-    </xacro:include>
+    <xacro:include filename="$(find elite_description)/urdf/elite_description.urdf.xacro"/>
     <!-- Import control_xacro -->
-    <xacro:include filename="ec66.ros2_control.xacro" />
+    <xacro:include filename="ec66.ros2_control.xacro"/>
     <xacro:ec66_ros2_control name="FakeSystem" initial_positions_file="$(arg initial_positions_file)"/>
 </robot>

Commit message: Updated urdf names in launch files, changed spwan entity names, and ros2 control controller names, Tested moveit in humble

File: elite_description/urdf/elite_description.urdf.xacro (robot description, xacro)
@@ -4,5 +4,4 @@
     <xacro:arg name="use_gazebo" default="false"/>
     <xacro:arg name="arm" default="ec66"/>
-    <xacro:arg name="use_moveit" default="false"/>
     <!-- Include macros -->
     <xacro:include filename="$(find elite_description)/urdf/macro/elite_macro.xacro" />
@@ -25,9 +24,7 @@
         <origin xyz="0 0 0" rpy="0 0 0" />
     </xacro:elite_robot>
-    <xacro:unless value="$(arg use_moveit)">
-        <!-- Include ros2_control configuration for simulation -->
-        <xacro:if value="$(arg use_gazebo)">
-            <xacro:include filename="$(find elite_description)/urdf/elite_gazebo_ros2_control.urdf.xacro" />
-        </xacro:if>
-    </xacro:unless>
+    <!-- Include ros2_control configuration for simulation -->
+    <xacro:if value="$(arg use_gazebo)">
+        <xacro:include filename="$(find elite_description)/urdf/elite_gazebo_ros2_control.urdf.xacro" />
+    </xacro:if>
 </robot>

File: elite_description/urdf/macro/elite_common.xacro (robot description, xacro)
@@ -3,12 +3,12 @@
   <!-- Load parameters from YAML files -->
   <xacro:property
-    name="joint_limits_parameters"
-    value="${xacro.load_yaml('$(arg joint_limit_params_file)')}"/>
+      name="joint_limits_parameters"
+      value="${xacro.load_yaml('$(arg joint_limit_params_file)')}"/>
   <xacro:property
-    name="joint_origins_parameters"
-    value="${xacro.load_yaml('$(arg joint_origin_params_file)')}"/>
+      name="joint_origins_parameters"
+      value="${xacro.load_yaml('$(arg joint_origin_params_file)')}"/>
   <xacro:property
-    name="link_inertials_parameters"
-    value="${xacro.load_yaml('$(arg link_inertials_params_file)')}"/>
+      name="link_inertials_parameters"
+      value="${xacro.load_yaml('$(arg link_inertials_params_file)')}"/>
   <!-- Extract subsections from yaml dictionaries -->
   <xacro:property name="joint_limits" value="${joint_limits_parameters['joint_limits']}"/>
@@ -17,51 +17,51 @@
   <!-- Define macros using loaded parameters -->
   <xacro:macro name="link_macro" params="name">
-    <link name="${name}">
-      <inertial>
-        <origin
-            xyz="
-                ${link_inertials[name]['origin']['x']}
-                ${link_inertials[name]['origin']['y']}
-                ${link_inertials[name]['origin']['z']}
-                "
-            rpy="0 0 0" />
-        <mass value="${link_inertials[name]['mass']}" />
-        <inertia
-            ixx="${link_inertials[name]['inertia']['ixx']}"
-            ixy="${link_inertials[name]['inertia']['ixy']}"
-            ixz="${link_inertials[name]['inertia']['ixz']}"
-            iyy="${link_inertials[name]['inertia']['iyy']}"
-            iyz="${link_inertials[name]['inertia']['iyz']}"
-            izz="${link_inertials[name]['inertia']['izz']}" />
-      </inertial>
-      <visual>
-        <origin xyz="0 0 0" rpy="0 0 0" />
-        <geometry>
-          <mesh filename="package://elite_description/meshes/ec66/${name}.stl" />
-        </geometry>
-      </visual>
-      <collision>
-        <origin xyz="0 0 0" rpy="0 0 0" />
-        <geometry>
-          <mesh filename="package://elite_description/meshes/ec66/${name}.stl" />
-        </geometry>
-      </collision>
-    </link>
+      <link name="${name}">
+          <inertial>
+              <origin
+                  xyz="
+                      ${link_inertials[name]['origin']['x']}
+                      ${link_inertials[name]['origin']['y']}
+                      ${link_inertials[name]['origin']['z']}
+                      "
+                  rpy="0 0 0" />
+              <mass value="${link_inertials[name]['mass']}" />
+              <inertia
+                  ixx="${link_inertials[name]['inertia']['ixx']}"
+                  ixy="${link_inertials[name]['inertia']['ixy']}"
+                  ixz="${link_inertials[name]['inertia']['ixz']}"
+                  iyy="${link_inertials[name]['inertia']['iyy']}"
+                  iyz="${link_inertials[name]['inertia']['iyz']}"
+                  izz="${link_inertials[name]['inertia']['izz']}" />
+          </inertial>
+          <visual>
+              <origin xyz="0 0 0" rpy="0 0 0" />
+              <geometry>
+                  <mesh filename="package://elite_description/meshes/ec66/${name}.stl" />
+              </geometry>
+          </visual>
+          <collision>
+              <origin xyz="0 0 0" rpy="0 0 0" />
+              <geometry>
+                  <mesh filename="package://elite_description/meshes/ec66/${name}.stl" />
+              </geometry>
+          </collision>
+      </link>
   </xacro:macro>
   <xacro:macro name="joint_macro" params="name">
-    <joint name="${name}" type="revolute">
-      <origin
-        xyz="${joint_origins[name]['origin_xyz']}"
-        rpy="${joint_origins[name]['origin_rpy']}" />
-      <parent link="${joint_origins[name]['parent']}" />
-      <child link="${joint_origins[name]['child']}" />
-      <axis xyz="0 0 1" />
-      <limit
-        lower="${joint_limits[name]['lower']}"
-        upper="${joint_limits[name]['upper']}"
-        effort="${joint_limits[name]['effort']}"
-        velocity="${joint_limits[name]['velocity']}" />
-      <dynamics damping="1.5" friction="3.5" />
-    </joint>
+      <joint name="${name}" type="revolute">
+          <origin
+              xyz="${joint_origins[name]['origin_xyz']}"
+              rpy="${joint_origins[name]['origin_rpy']}" />
+          <parent link="${joint_origins[name]['parent']}" />
+          <child link="${joint_origins[name]['child']}" />
+          <axis xyz="0 0 1" />
+          <limit
+              lower="${joint_limits[name]['lower']}"
+              upper="${joint_limits[name]['upper']}"
+              effort="${joint_limits[name]['effort']}"
+              velocity="${joint_limits[name]['velocity']}" />
+          <dynamics damping="1.5" friction="3.5" />
+      </joint>
   </xacro:macro>
 </robot>

File: elite_moveit/config/ec66.urdf.xacro (robot description, xacro)
@@ -1,11 +1,7 @@
 <?xml version="1.0"?>
-<robot xmlns:xacro="http://www.ros.org/wiki/xacro" name="ec66">
+<robot xmlns:xacro="http://www.ros.org/wiki/xacro" name="elite">
     <xacro:arg name="initial_positions_file" default="initial_positions.yaml" />
     <xacro:arg name="arm" default="ec66"/>
-    <xacro:arg name="use_moveit" default="true"/>
-    <!-- Import elite_description urdf file with arm_type argument -->
+    <!-- Import elite_description urdf file with arm argument -->
     <xacro:include filename="$(find elite_description)/urdf/elite_description.urdf.xacro"/>
-    <!-- Import control_xacro -->
-    <xacro:include filename="ec66.ros2_control.xacro" />
-    <xacro:ec66_ros2_control name="FakeSystem" initial_positions_file="$(arg initial_positions_file)"/>
 </robot>

File: elite_moveit/config/ec66_simulation.urdf.xacro (robot description, xacro)
@@ -1,11 +1,8 @@
 <?xml version="1.0"?>
-<robot xmlns:xacro="http://www.ros.org/wiki/xacro" name="ec66">
+<robot xmlns:xacro="http://www.ros.org/wiki/xacro" name="elite">
     <xacro:arg name="initial_positions_file" default="initial_positions.yaml" />
-    <xacro:arg name="use_gazebo" value="true"/>
-    <xacro:arg name="arm" value="ec66"/>
-    <!-- Import ec66 urdf file with use_gazebo set to true -->
+    <xacro:arg name="use_gazebo" default="true"/>
+    <xacro:arg name="arm" default="ec66"/>
+    <!-- Import ec66 urdf file with use_gazebo set to true and arm argument-->
     <xacro:include filename="$(find elite_description)/urdf/elite_description.urdf.xacro"/>
-    <!-- Import control_xacro -->
-    <xacro:include filename="ec66.ros2_control.xacro"/>
-    <xacro:ec66_ros2_control name="FakeSystem" initial_positions_file="$(arg initial_positions_file)"/>
 </robot>

Commit message: Refactored moveit simulation launch files, updated xacro

File: elite_description/urdf/elite_description.urdf.xacro (robot description, xacro)
@@ -1,35 +1,40 @@
 <?xml version="1.0"?>
+<!--
+Author: Pradheep Padmanabhan
+Contributor: Adarsh Karan K P
+-->
 <robot xmlns:xacro="http://www.ros.org/wiki/xacro" name="elite">
-    <!-- Set use_gz = true for Modern Gazebo -->
-    <xacro:arg name="use_gz" default="false"/>
-    <xacro:arg name="arm_type" default="ec66"/>
-    <!-- Include macros -->
-    <xacro:include filename="$(find elite_description)/urdf/macro/elite_macro.xacro" />
-    <!-- Elite arm parameters -->
-    <xacro:arg name="arm_parent" default="world"/>
-    <xacro:arg name="tf_prefix" default=""/>
-    <xacro:arg name="joint_limit_params_file" default="$(find elite_description)/config/$(arg arm_type)/joint_limits.yaml"/>
-    <xacro:arg name="kinematics_params_file" default="$(find elite_description)/config/$(arg arm_type)/kinematics.yaml"/>
-    <xacro:arg name="physical_params_file" default="$(find elite_description)/config/$(arg arm_type)/physical_parameters.yaml"/>
-    <xacro:arg name="initial_joint_positions_file" default="$(find elite_description)/config/$(arg arm_type)/initial_positions.yaml"/>
-    <!-- Load parameters from YAML file -->
-    <xacro:property
-        name="elite_initial_positions"
-        value="${xacro.load_yaml('$(arg initial_joint_positions_file)')}"
+<!-- This is the main URDF file for ec66 elite arm-->
+  <!-- Set use_gz = true for Modern Gazebo Simulation-->
+  <xacro:arg name="use_gz" default="false"/>
+  <xacro:arg name="arm_type" default="ec66"/>
+  <!-- Include macros -->
+  <xacro:include filename="$(find elite_description)/urdf/xacros/elite_macro.xacro" />
+  <!-- Elite arm parameters -->
+  <xacro:arg name="arm_parent" default="world"/>
+  <xacro:arg name="tf_prefix" default=""/>
+  <xacro:arg name="joint_limit_params_file" default="$(find elite_description)/config/$(arg arm_type)/joint_limits.yaml"/>
+  <xacro:arg name="kinematics_params_file" default="$(find elite_description)/config/$(arg arm_type)/kinematics.yaml"/>
+  <xacro:arg name="physical_params_file" default="$(find elite_description)/config/$(arg arm_type)/physical_parameters.yaml"/>
+  <xacro:arg name="initial_joint_positions_file" default="$(find elite_description)/config/$(arg arm_type)/initial_positions.yaml"/>
+  <!-- Load parameters from YAML file -->
+  <xacro:property
+    name="elite_initial_positions"
+    value="${xacro.load_yaml('$(arg initial_joint_positions_file)')}"
     />
-    <!-- Create arm -->
-    <xacro:elite_robot
-        name="$(arg arm_type)"
-        tf_prefix="$(arg tf_prefix)"
-        parent="$(arg arm_parent)"
-        joint_limits_parameters_file="$(arg joint_limit_params_file)"
-        kinematics_parameters_file="$(arg kinematics_params_file)"
-        physical_parameters_file="$(arg physical_params_file)"
+  <!-- Create arm -->
+  <xacro:elite_robot
+    name="$(arg arm_type)"
+    tf_prefix="$(arg tf_prefix)"
+    parent="$(arg arm_parent)"
+    joint_limits_parameters_file="$(arg joint_limit_params_file)"
+    kinematics_parameters_file="$(arg kinematics_params_file)"
+    physical_parameters_file="$(arg physical_params_file)"
     >
-        <origin xyz="0 0 0" rpy="0 0 0" />
-    </xacro:elite_robot>
-    <!-- Include ros2_control configuration for simulation -->
-    <xacro:if value="$(arg use_gz)">
-        <xacro:include filename="$(find elite_description)/urdf/elite_gz_ros2_control.urdf.xacro" />
-    </xacro:if>
+    <origin xyz="0 0 0" rpy="0 0 0" />
+  </xacro:elite_robot>
+  <!-- Include ros2_control configuration for simulation -->
+  <xacro:if value="$(arg use_gz)">
+    <xacro:include filename="$(find elite_description)/urdf/xacros/elite_gz_ros2_control.urdf.xacro" />
+  </xacro:if>
 </robot>
